File: pcb/macropad.kicad_sch (KiCad schematic)
At the start: 53 parts, among them SW1 SW_Push, SW10 SW_Push, SW11 SW_Push, SW12 SW_Push, SW13 RotaryEncoder_Switch, SW14 RotaryEncoder_Switch, SW15 SW_Push, SW16 SW_Push, SW2 SW_Push, SW3 SW_Push, SW4 SW_Push, SW5 SW_Push, SW6 SW_Push, SW7 SW_Push, SW8 SW_Push, SW9 SW_Push, U1 XIAO-RP2040-DIP, U3 MCP23S17_SO

Commit message: 2
Parts:
- removed D13, D14: D, Diode_THT:D_DO-35_SOD27_P7.62mm_Horizontal, symbol Device:D
- removed D30, D31: SK6812MINI, LED_SMD:LED_SK6812MINI_PLCC4_3.5x3.5mm_P1.75mm, symbol LED:SK6812MINI
- removed SW14: RotaryEncoder_Switch, Rotary_Encoder:RotaryEncoder_Alps_EC11E-Switch_Vertical_H20mm_CircularMountingHoles, symbol Device:RotaryEncoder_Switch
- removed SW15, SW16: SW_Push, Button_Switch_Keyboard:SW_Cherry_MX_1.00u_PCB, symbol Switch:SW_Push
- removed U3: MCP23S17_SO, Package_SO:SOIC-28W_7.5x17.9mm_P1.27mm, symbol Interface_Expansion:MCP23S17_SO
- added R3, R4: R, Resistor_THT:R_Axial_DIN0204_L3.6mm_D1.6mm_P7.62mm_Horizontal, symbol Device:R
- added U2: MCP23017_SO, Package_SO:SOIC-28W_7.5x17.9mm_P1.27mm, symbol Interface_Expansion:MCP23017_SO
- D100, D15, D16, D17, D18, D19, D20, D21, D22, D23, D24, D25, D26, D27, D28, D29: footprint LED_SMD:LED_SK6812MINI_PLCC4_3.5x3.5mm_P1.75mm -> led:SK6812MINI-E
Connections:
- net +3.3V: now also R3.2, R4.2, U2.18 (~{RESET}), U2.9 (VDD)
- net GND: now also U2.10 (VSS), U2.15 (A0), U2.16 (A1), U2.17 (A2)
- net at SW13.S1: now also U1.2 (GPIO27/ADC1/A1)
- net at D12.1 (K), D4.1 (K), D8.1 (K): now also U2.4 (GPB3)
- net at U1.1 (GPIO26/ADC0/A0): now also SW13.S2
- net at U1.3 (GPIO28/ADC2/A2): now also SW13.A
- net at U1.4 (GPIO29/ADC3/A3): now also SW13.B
- net at Brd1.4 (SDA), R2.1, U1.5 (GPIO6/SDA): now also R3.1, U2.13 (SDA)
- net at Brd1.3 (SCL), R1.1, U1.6 (GPIO7/SCL): now also R4.1, U2.12 (SCK)
- net at U1.7 (GPIO0/TX): no longer D100.3 (DIN)
- net at SW5.1, SW6.1, SW7.1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: now also U2.6 (GPB5)
- net at SW1.1, SW2.1, SW3.1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: now also U2.5 (GPB4)
- net at D10.1 (K), D2.1 (K), D6.1 (K): now also U2.2 (GPB1)
- net at D1.1 (K), D5.1 (K), D9.1 (K): now also U2.1 (GPB0)
- net at D11.1 (K), D3.1 (K), D7.1 (K): now also U2.3 (GPB2); no longer SW13.S2
- net at SW10.1, SW11.1, SW12.1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: now also U2.7 (GPB6)
- new net: D100.3 (DIN), U2.8 (GPB7)
Other:
- moved on the sheet: SW13
